File: KiCad_Files/KiCad/MosaicTimeSync/MosaicTimeSync.kicad_sch (KiCad schematic)
At the start: 1 part

Commit message: KiCad update
Other:
- title: M2_mosaic G5-T_Module  -> MosaicTimeSync
Changed lines of the file:
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@@
 	(paper "A3")
 	(title_block
-		(title "M2_mosaic G5-T_Module ")
+		(title "MosaicTimeSync")
 		(date "2025-09-02")
 		(rev "01")
 		(company "Septentrio")
+		(comment 2 "under the Fundamental Elements Grant EUSPA/GRANT/02/2024")
+		(comment 3 "co-funded by the European Union Agency for the Space Programme ")
+		(comment 4 "MosaicTimeSync project has been documented by Septentrio")
 	)
 	(text "CHANGE LOG"

Commit message: HW files update
Other:
- note added: "M.2 Key B with Mosaic G5 GNSS Module"
- note added: "Project: MosaicTimeSync Varient: mosaic-G5 T"
- note added: "Ultra-compact high-precision GNSS time synchronization receiver"
- note added: "mosaic-G5 T"
