File: KiCad_Files/KiCad/MosaicTimeSync/M2_Edge connector.kicad_sch (KiCad schematic)
At the start: 11 parts, among them Q2 NTK3043NT1G

Commit message: KiCad update
Other:
- note added: "Fiducials"
- note added: "M.2 Key B"
- title: M2_mosaic G5-T_Module  -> MosaicTimeSync
- moved on the sheet: C3, FID1, FID2, FID3, FID4, FID5, FID6, J2, Q2, R5, R6

Commit message: HW files update
Parts:
- renumbered C3 to C?, FID5 to FID?, FID6 to FID?, FID1 to FID?, FID2 to FID?, FID4 to FID?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

Commit message: Septentrio logo
Parts:
- gave numbers to parts that had none: 11
