File: KiCad_Files/KiCad/MosaicTimeSync/mosaic-G5.kicad_sch (KiCad schematic)
At the start: 14 parts, among them J1 U.FL-R-SMT_10_, U1 mosaic-G5 T, Y1 RV-3032-C7

Commit message: KiCad update
Other:
- note added: "Antenna"
- note added: "Mosaic-G5 T"
- title: M2_mosaic G5-T_Module  -> MosaicTimeSync
- moved on the sheet: C1, C2, C5, D1, D2, J1, R1, R12, R13, R4, R7, R8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

Commit message: HW files update
Parts:
- renumbered C1 to C?, C2 to C?, C5 to C?, D1 to D?, D2 to D?, J1 to J?, R12 to R?, R7 to R?, R1 to R?, R13 to R?, R4 to R?, R8 to R?, U1 to U?, Y1 to Y?
Connections:
- net +3.3V: now also U?.16 (RESERVED), U?.18 (RESERVED); no longer U?.44 (VDD_3V3), U?.45 (VDD_3V3)
- net GND: now also U?.10 (TXD1), U?.12 (USB_DP), U?.13 (USB_DN), U?.14 (USB_VBUS), U?.15 (RESERVED), U?.19 (RESERVED), U?.2 (ANT_1), U?.20 (RESERVED), U?.22 (RESERVED), U?.23 (RESERVED), U?.24 (RESERVED), U?.25 (TXD2), U?.26 (NRTS2), U?.28 (NCTS2), U?.29 (RXD2), U?.30 (RESERVED), U?.31 (RESERVED), U?.32 (RESERVED), U?.33 (RESERVED), U?.35 (RESERVED), U?.36 (RESERVED), U?.37 (RESERVED), U?.38 (RESERVED), U?.39 (EVENTA), U?.40 (EVENTB), U?.42 (PPS1), U?.43 (PPS2), U?.47 (REF_O), U?.48 (REF_I), U?.5 (RESERVED), U?.50 (VREF_I), U?.51 (VREF_O), U?.52 (GPIO1), U?.53 (GPIO2), U?.54 (VANT), U?.7 (NRST_IN), U?.8 (RESERVED), U?.9 (RXD1); no longer U?.1 (GND), U?.11 (GND), U?.17 (GND), U?.21 (GND), U?.27 (GND), U?.3 (GND), U?.34 (GND), U?.4 (GND), U?.41 (GND), U?.46 (GND), U?.49 (GND), U?.55 (GND), U?.56 (GND), U?.57 (GND), U?.58 (GND), U?.59 (GND), U?.6 (GND), U?.60 (GND), U?.61 (GND), U?.62 (GND), U?.63 (GND), U?.64 (GND), U?.65 (GND), U?.66 (GND), U?.67 (GND), U?.68 (GND), U?.69 (GND), U?.70 (GND), U?.71 (GND), U?.72 (GND), U?.73 (GND), U?.74 (GND), U?.75 (GND), U?.76 (GND), U?.77 (GND), U?.78 (GND), U?.79 (GND), U?.80 (GND), U?.81 (GND), U?.82 (GND), U?.83 (GND), U?.84 (GND), U?.85 (GND), U?.86 (GND), U?.87 (GND), U?.88 (GND), U?.89 (GND), U?.90 (GND), U?.91 (GND), U?.92 (GND), U?.93 (GND), U?.94 (GND)

Commit message: Septentrio logo
Parts:
- gave numbers to parts that had none: 14
Connections:
- net +3.3V: now also U1.44 (VDD_3V3), U1.45 (VDD_3V3); no longer U1.16 (RESERVED), U1.18 (RESERVED)
- net GND: now also U1.1 (GND), U1.11 (GND), U1.17 (GND), U1.21 (GND), U1.27 (GND), U1.3 (GND), U1.34 (GND), U1.4 (GND), U1.41 (GND), U1.46 (GND), U1.49 (GND), U1.55 (GND), U1.56 (GND), U1.57 (GND), U1.58 (GND), U1.59 (GND), U1.6 (GND), U1.60 (GND), U1.61 (GND), U1.62 (GND), U1.63 (GND), U1.64 (GND), U1.65 (GND), U1.66 (GND), U1.67 (GND), U1.68 (GND), U1.69 (GND), U1.70 (GND), U1.71 (GND), U1.72 (GND), U1.73 (GND), U1.74 (GND), U1.75 (GND), U1.76 (GND), U1.77 (GND), U1.78 (GND), U1.79 (GND), U1.80 (GND), U1.81 (GND), U1.82 (GND), U1.83 (GND), U1.84 (GND), U1.85 (GND), U1.86 (GND), U1.87 (GND), U1.88 (GND), U1.89 (GND), U1.90 (GND), U1.91 (GND), U1.92 (GND), U1.93 (GND), U1.94 (GND); no longer U1.10 (TXD1), U1.12 (USB_DP), U1.13 (USB_DN), U1.14 (USB_VBUS), U1.15 (RESERVED), U1.19 (RESERVED), U1.2 (ANT_1), U1.20 (RESERVED), U1.22 (RESERVED), U1.23 (RESERVED), U1.24 (RESERVED), U1.25 (TXD2), U1.26 (NRTS2), U1.28 (NCTS2), U1.29 (RXD2), U1.30 (RESERVED), U1.31 (RESERVED), U1.32 (RESERVED), U1.33 (RESERVED), U1.35 (RESERVED), U1.36 (RESERVED), U1.37 (RESERVED), U1.38 (RESERVED), U1.39 (EVENTA), U1.40 (EVENTB), U1.42 (PPS1), U1.43 (PPS2), U1.47 (REF_O), U1.48 (REF_I), U1.5 (RESERVED), U1.50 (VREF_I), U1.51 (VREF_O), U1.52 (GPIO1), U1.53 (GPIO2), U1.54 (VANT), U1.7 (NRST_IN), U1.8 (RESERVED), U1.9 (RXD1)
