File: KiCad_Files/KiCad/moTi/moTi.kicad_pcb (KiCad board)
At the start: 4 copper layers, 22 x 42 mm, 38 parts, among them J1 U.FL-R-SMT_10_, Q1 NTK3139PT5G, Q2 NTK3043NT1G, U1 mosaic-G5 T, U2 TLV3511DCKR, U5 SN74LVC1G3157DRLR, Y1 RV-3032-C7

Commit message: kicad file clean up
Parts:
- removed C7: 1.0n, Capacitor_SMD:C_0402_1005Metric
- added R14: 10k, Resistor_SMD:R_0402_1005Metric, F.Cu at (92.2, 108.7)
- R2: value 2.2k -> 1.5k
- moved R11 0.22 mm to (94.9, 104.5)
- moved U2 0.22 mm to (93.4, 106.3)
- moved C8 0.22 mm to (92.5, 104.4)
- moved Q1 0.18 mm to (93.8, 108.7)
Connections:
- R2 pad 1: Net-(C7-Pad2) -> CLK_10M_IN
Routing:
- net GND: track 29.8 -> 34.9 mm
- net CLK_10M_IN: track 9.14 -> 11.1 mm
- net Ref_CLK_SEL: track 41.8 -> 43.0 mm
- net VREF_O: track 16.2 -> 17.4 mm
- net Net-(C7-Pad2): track 0.92 -> 0.00 mm
- net UART_TX: track 21.0 -> 21.8 mm
- net +3.3V: track 15.7 -> 16.5 mm
Other:
- outline, holes or cut-outs redrawn
- board text added: "-"
- board text added: "180"
- board text added: "200"
- board text added: "220"
- board text added: "50 +/- 10%"
- board text added: "90 +/- 10%"
- board text added: "BOTTOM"
- board text added: "Coplanar Waveguide"
- board text added: "Coplanar spacing"
- board text added: "DIFF"
- board text added: "Designed [um]"
- board text added: "Impedance [Ohm]"
- board text added: "L02"
- board text added: "L03"
- board text added: "Layer"
- board text added: "Ref Layer Lower"
- board text added: "Ref Layer Upper"
- board text added: "TOP"
- board text added: "Target [Ohm] & Tolerance [%]"
- board text added: "Trace spacing {dblquote}Airgap{dblquote}"
- board text added: "Trace width"

Commit message: general clean up
Parts:
- removed C5: 100n, Capacitor_SMD:C_0402_1005Metric
- removed R12, R13: 10k, Resistor_SMD:R_0402_1005Metric
- removed R5, R6: 0, Resistor_SMD:R_0402_1005Metric
- removed R7, R8: 4k7, Resistor_SMD:R_0402_1005Metric
- removed Y1: RV-3032-C7, rv-3032-c7:RV3032C7
Connections:
- J2 pad 2: VBAT -> unconnected-(J2-3.3V/VBAT-Pad2)
- J2 pad 4: VBAT -> unconnected-(J2-3.3V/VBAT-Pad4)
- J2 pad 40: Net-(J2-SMB_CLK) -> unconnected-(J2-SMB_CLK-Pad40)
- J2 pad 42: Net-(J2-SMB_DATA) -> unconnected-(J2-SMB_DATA-Pad42)
- U1 pad 30: SCL -> unconnected-(U1A-RESERVED-Pad30)
- U1 pad 31: SDA -> unconnected-(U1A-RESERVED-Pad31)
Routing:
- net SCL: track 18.7 -> 0.00 mm, vias 3 -> 0
- net SDA: track 15.4 -> 0.00 mm, vias 2 -> 0
- net Net-(J2-SMB_DATA): track 9.65 -> 0.00 mm, vias 1 -> 0
- net VBAT: track 8.72 -> 0.00 mm, vias 1 -> 0
- net Net-(J2-SMB_CLK): track 7.89 -> 0.00 mm, vias 1 -> 0
- net +3.3V: track 16.5 -> 14.1 mm, vias 12 -> 10
- net Net-(Y1-VBACKUP): track 1.66 -> 0.00 mm
- net Net-(Y1-EVI): track 1.04 -> 0.00 mm
