File: KiCad_Files/KiCad/moTi/moTi.kicad_sch (KiCad schematic)
At the start: 1 part

Commit message: HW file update
Other:
- note added: "Project: moTi Varient: mosaic-G5 T"
- note removed: "Project: MosaicTimeSync Varient: mosaic-G5 T"
- title: MosaicTimeSync -> moTi
Changed lines of the file:
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@@
 	(paper "A3")
 	(title_block
-		(title "MosaicTimeSync")
+		(title "moTi")
 		(date "2025-09-02")
 		(rev "01")
@@
 		(comment 2 "Programme under the Fundamental Elements")
 		(comment 3 "co-funded by the European Union Agency for the Space")
-		(comment 4 "MosaicTimeSync project has been documented by Septentrio")
-	)
-	(text "Project: 			MosaicTimeSync\nVarient: 			mosaic-G5 T"
+		(comment 4 "moTi project has been documented by Septentrio")
+	)
+	(text "Project: 			moTi\nVarient: 			mosaic-G5 T"
 		(exclude_from_sim no)
 		(at 110.49 99.822 0)
@@
 		)
 		(instances
-			(project "MosaicTimeSync"
+			(project "moTi"
 				(path "/a9fd92c2-3c56-4e0a-a5ac-af47c0a80946"
 					(page "4")
@@
 		)
 		(instances
-			(project "MosaicTimeSync"
+			(project "moTi"
 				(path "/a9fd92c2-3c56-4e0a-a5ac-af47c0a80946"
 					(page "2")
@@
 		)
 		(instances
-			(project "MosaicTimeSync"
+			(project "moTi"
 				(path "/a9fd92c2-3c56-4e0a-a5ac-af47c0a80946"
 					(page "3")

Commit message: I2C change
Parts:
- PCB1: value ~ -> (none)

Commit message: general clean up
Changed lines of the file:
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@@
 		(title "moTi")
 		(date "2025-09-02")
-		(rev "01")
+		(rev "02")
 		(company "Septentrio")
 		(comment 1 "Grant EUSPA/GRANT/02/2024")
@@
 		(comment 3 "co-funded by the European Union Agency for the Space")
 		(comment 4 "moTi project has been documented by Septentrio")
+		(comment 5 "   ")
 	)
 	(text "Project: 			moTi\nVarient: 			mosaic-G5 T"
@@
 		)
 	)
+	(text_box "Schematics arranged by Laetitia.K"
+		(exclude_from_sim no)
+		(at 372.11 271.6417 0)
+		(size 35.56 3.9483)
+		(margins 0.9525 0.9525 0.9525 0.9525)
+		(stroke
+			(width -0.0001)
+			(type solid)
+		)
+		(fill
+			(type none)
+		)
+		(effects
+			(font
+				(size 1.27 1.27)
+				(color 132 0 0 1)
+			)
+			(justify left top)
+		)
+	)
 	(polyline
 		(pts
@@
 	)
 	(image
-		(at 389.89 260.35)
+		(at 387.35 260.35)
 		(scale 0.614071)
 		(data "iVBORw0KGgoAAAANSUhEUgAAAREAAABcCAYAAABJJYGIAAAAAXNSR0IArs4c6QAAAARnQU1BAACx"
@@
 		)
 		(column_widths 54.61 54.61 78.74 95.25)
-		(row_heights 7.366 8.636)
+		(row_heights 7.366 8.636 8.636)
 		(cells
 			(table_cell "Revision"
@@
 				(size 95.25 8.636)
 				(margins 0.9525 0.9525 0.9525 0.9525)
+				(span 1 1)
+				(fill
+					(type none)
+				)
+				(effects
+					(font
+						(size 2.54 2.54)
+					)
+					(justify left top)
+				)
+			)
+			(table_cell "02"
+				(exclude_from_sim no)
+				(at 58.928 165.862 0)
+				(size 54.61 8.636)
+				(margins 0.9525 0.9525 0.9525 0.9525)
+				(span 1 1)
+				(fill
+					(type none)
+				)
+				(effects
+					(font
+						(size 2.54 2.54)
+					)
+					(justify left top)
+				)
+			)
+			(table_cell "2026-04-15"
+				(exclude_from_sim no)
+				(at 113.538 165.862 0)
+				(size 54.61 8.636)
+				(margins 0.9525 0.9525 0.9525 0.9525)
+				(span 1 1)
+				(fill
+					(type none)
+				)
+				(effects
+					(font
+						(size 2.54 2.54)
+					)
+					(justify left top)
+				)
+			)
+			(table_cell "K. Heyndrick"
+				(exclude_from_sim no)
+				(at 168.148 165.862 0)
+				(size 78.74 8.636)
+				(margins 0.9525 0.9525 0.9525 0.9525)
+				(span 1 1)
+				(fill
+					(type none)
+				)
+				(effects
+					(font
+						(size 2.54 2.54)
+					)
+					(justify left top)
+				)
+			)
+			(table_cell "Update:Add pull-down resisitor on gate Q1"
+				(exclude_from_sim no)
+				(at 246.888 165.862 0)
+				(size 95.25 8.636)
+				(margins 0.9525 0.9525 0.9525 0.9525)
