File: KiCad_Files/KiCad/moTi/mosaic-G5.kicad_sch (KiCad schematic)
At the start: 14 parts, among them J1 U.FL-R-SMT_10_, U1 mosaic-G5 T, Y1 RV-3032-C7

Commit message: HW file update
Parts:
- renumbered C1 to C?, C2 to C?, C5 to C?, D1 to D?, D2 to D?, J1 to J?, R12 to R?, R7 to R?, R1 to R?, R13 to R?, R4 to R?, R8 to R?, U1 to U?, Y1 to Y?
Connections:
- net +3.3V: now also U?.16 (RESERVED), U?.18 (RESERVED); no longer U?.44 (VDD_3V3), U?.45 (VDD_3V3)
- net GND: now also U?.10 (TXD1), U?.12 (USB_DP), U?.13 (USB_DN), U?.14 (USB_VBUS), U?.15 (RESERVED), U?.19 (RESERVED), U?.2 (ANT_1), U?.20 (RESERVED), U?.22 (RESERVED), U?.23 (RESERVED), U?.24 (RESERVED), U?.25 (TXD2), U?.26 (NRTS2), U?.28 (NCTS2), U?.29 (RXD2), U?.30 (RESERVED), U?.31 (RESERVED), U?.32 (RESERVED), U?.33 (RESERVED), U?.35 (RESERVED), U?.36 (RESERVED), U?.37 (RESERVED), U?.38 (RESERVED), U?.39 (EVENTA), U?.40 (EVENTB), U?.42 (PPS1), U?.43 (PPS2), U?.47 (REF_O), U?.48 (REF_I), U?.5 (RESERVED), U?.50 (VREF_I), U?.51 (VREF_O), U?.52 (GPIO1), U?.53 (GPIO2), U?.54 (VANT), U?.7 (NRST_IN), U?.8 (RESERVED), U?.9 (RXD1); no longer U?.1 (GND), U?.11 (GND), U?.17 (GND), U?.21 (GND), U?.27 (GND), U?.3 (GND), U?.34 (GND), U?.4 (GND), U?.41 (GND), U?.46 (GND), U?.49 (GND), U?.55 (GND), U?.56 (GND), U?.57 (GND), U?.58 (GND), U?.59 (GND), U?.6 (GND), U?.60 (GND), U?.61 (GND), U?.62 (GND), U?.63 (GND), U?.64 (GND), U?.65 (GND), U?.66 (GND), U?.67 (GND), U?.68 (GND), U?.69 (GND), U?.70 (GND), U?.71 (GND), U?.72 (GND), U?.73 (GND), U?.74 (GND), U?.75 (GND), U?.76 (GND), U?.77 (GND), U?.78 (GND), U?.79 (GND), U?.80 (GND), U?.81 (GND), U?.82 (GND), U?.83 (GND), U?.84 (GND), U?.85 (GND), U?.86 (GND), U?.87 (GND), U?.88 (GND), U?.89 (GND), U?.90 (GND), U?.91 (GND), U?.92 (GND), U?.93 (GND), U?.94 (GND)
Other:
- title: MosaicTimeSync -> moTi
Changed lines of the file:
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@@
 	(paper "A3")
 	(title_block
-		(title "MosaicTimeSync")
+		(title "moTi")
 		(date "2025-09-02")
 		(rev "01")
@@
 		(comment 2 "Programme under the Fundamental Elements")
 		(comment 3 "co-funded by the European Union Agency for the Space ")
-		(comment 4 "MosaicTimeSync project has been documented by Septentrio")
+		(comment 4 "moTi project has been documented by Septentrio")
 	)
 	(rectangle
@@
 				)
 				(justify right)
+				(hide yes)
 			)
 		)
@@
 				)
 				(justify left)
+				(hide yes)
 			)
 		)
@@
 				)
 				(justify right)
+				(hide yes)
 			)
 		)
@@
 				)
 				(justify left)
+				(hide yes)
 			)
 		)
@@
 				)
 				(justify left)
+				(hide yes)
 			)
 		)
@@
 				)
 				(justify left)
+				(hide yes)
 			)
 		)
@@
 				)
 				(justify right)
+				(hide yes)
 			)
 		)
@@
 				)
 				(justify left)
+				(hide yes)
 			)
 		)
@@
 				)
 				(justify right)
+				(hide yes)
 			)
 		)
@@
 				)
 				(justify right)
+				(hide yes)
 			)
 		)
@@
 				)
 				(justify left)
+				(hide yes)
 			)
 		)
@@
 				)
 				(justify right)
+				(hide yes)
 			)
 		)
@@
 				)
 				(justify left)
+				(hide yes)
 			)
 		)
@@
 				)
 				(justify right)
+				(hide yes)
 			)
 		)
@@
 				)
 				(justify left)
+				(hide yes)
 			)
 		)
@@
 		(on_board yes)
 		(dnp no)
-		(property "Reference" "R12"
+		(property "Reference" "R?"
 			(at 290.83 84.328 90)
 			(effects
@@
 		(dnp no)
 		(fields_autoplaced yes)
-		(property "Reference" "#PWR02"
+		(property "Reference" "#PWR?"
 			(at 78.74 228.6 0)
 			(effects
@@
 		(dnp no)
 		(fields_autoplaced yes)
-		(property "Reference" "D1"
+		(property "Reference" "D?"
 			(at 191.4525 64.77 0)
 			(effects
@@
 		(dnp no)
 		(fields_autoplaced yes)
-		(property "Reference" "R7"
+		(property "Reference" "R?"
 			(at 190.5 111.7599 0)
 			(effects
@@
 		(dnp no)
 		(fields_autoplaced yes)
-		(property "Reference" "#PWR037"
+		(property "Reference" "#PWR?"
 			(at 184.15 82.55 0)
 			(effects
@@
 		(dnp no)
 		(fields_autoplaced yes)
-		(property "Reference" "#PWR033"
+		(property "Reference" "#PWR?"
 			(at 187.96 111.76 0)
 			(effects
@@
 		(dnp no)
 		(fields_autoplaced yes)
-		(property "Reference" "#PWR034"
+		(property "Reference" "#PWR?"
 			(at 196.85 111.76 0)
 			(effects
@@
 		(dnp no)
 		(fields_autoplaced yes)
-		(property "Reference" "#PWR029"
+		(property "Reference" "#PWR?"
 			(at 78.74 95.25 0)
 			(effects
@@
 		(dnp no)
 		(fields_autoplaced yes)
-		(property "Reference" "U1"
+		(property "Reference" "U?"
 			(at 121.92 62.23 0)
 			(effects
@@
 		(dnp no)
 		(fields_autoplaced yes)
-		(property "Reference" "#PWR05"
+		(property "Reference" "#PWR?"
 			(at 59.69 194.31 0)
 			(effects
@@
 		(on_board yes)
 		(dnp no)
-		(property "Reference" "R1"
+		(property "Reference" "R?"
 			(at 172.466 75.438 90)
 			(effects
@@
 		(on_board yes)
 		(dnp no)
-		(property "Reference" "R13"
+		(property "Reference" "R?"
 			(at 316.23 61.468 90)
 			(effects
@@
 		(on_board yes)
 		(dnp no)
-		(property "Reference" "R4"
+		(property "Reference" "R?"
 			(at 281.178 162.814 90)
 			(effects
@@
 		(dnp no)
 		(fields_autoplaced yes)
-		(property "Reference" "#PWR07"
+		(property "Reference" "#PWR?"
 			(at 284.48 93.98 0)
 			(effects
@@
 		(on_board yes)
 		(dnp no)
-		(property "Reference" "#PWR039"
+		(property "Reference" "#PWR?"
 			(at 307.34 62.23 0)
 			(effects
@@
 		(dnp no)
 		(fields_autoplaced yes)
-		(property "Reference" "C1"
+		(property "Reference" "C?"
 			(at 53.34 180.3399 0)
 			(effects
@@
 		(dnp no)
 		(fields_autoplaced yes)
-		(property "Reference" "#PWR06"
+		(property "Reference" "#PWR?"
 			(at 270.51 214.63 0)
 			(effects
@@
 		(dnp no)
 		(fields_autoplaced yes)
-		(property "Reference" "#PWR040"
+		(property "Reference" "#PWR?"
 			(at 285.75 63.5 0)
 			(effects
@@
 		(dnp no)
 		(fields_autoplaced yes)
-		(property "Reference" "#PWR01"
+		(property "Reference" "#PWR?"
 			(at 44.45 175.26 0)
 			(effects
@@
 		(dnp no)
 		(fields_autoplaced yes)
-		(property "Reference" "#PWR031"
+		(property "Reference" "#PWR?"
 			(at 283.21 148.59 0)
 			(effects
@@
 		(dnp no)
 		(fields_autoplaced yes)
-		(property "Reference" "#PWR030"
+		(property "Reference" "#PWR?"
 			(at 283.21 175.26 0)
 			(effects
@@
 		(dnp no)
 		(fields_autoplaced yes)
-		(property "Reference" "#PWR08"
+		(property "Reference" "#PWR?"
 			(at 207.01 69.85 0)
 			(effects
@@
 		(lib_id "mosaic-G5-T:mosaic-G5_T")
 		(at 81.28 149.86 0)
-		(unit 2)
+		(unit 1)
 		(exclude_from_sim no)
 		(in_bom yes)
@@
 		(dnp no)
 		(fields_autoplaced yes)
-		(property "Reference" "U1"
+		(property "Reference" "U?"
 			(at 121.92 137.16 0)
 			(effects
@@
 		(dnp no)
 		(fields_autoplaced yes)
-		(property "Reference" "#PWR04"
+		(property "Reference" "#PWR?"
 			(at 49.53 194.31 0)
 			(effects
@@
 		(on_board yes)
 		(dnp no)
-		(property "Reference" "J1"
+		(property "Reference" "J?"
 			(at 285.75 213.36 0)
 			(effects
@@
 		(dnp no)
 		(fields_autoplaced yes)
-		(property "Reference" "#PWR043"
+		(property "Reference" "#PWR?"
 			(at 184.15 85.09 0)
 			(effects
@@
 		(dnp no)
 		(fields_autoplaced yes)
-		(property "Reference" "#PWR027"
+		(property "Reference" "#PWR?"
 			(at 177.8 76.2 0)
 			(effects
@@
 		(dnp no)
 		(fields_autoplaced yes)
-		(property "Reference" "C2"
+		(property "Reference" "C?"
 			(at 63.5 180.3399 0)
 			(effects
@@
 		(on_board yes)
 		(dnp no)
-		(property "Reference" "Y1"
+		(property "Reference" "Y?"
 			(at 316.23 70.358 0)
 			(effects
@@
 		(dnp no)
 		(fields_autoplaced yes)
-		(property "Reference" "D2"
+		(property "Reference" "D?"
 			(at 287.02 151.4474 90)
 			(effects
@@
 		(dnp no)
 		(fields_autoplaced yes)
-		(property "Reference" "#PWR03"
+		(property "Reference" "#PWR?"
 			(at 166.37 228.6 0)
 			(effects
@@
 		(on_board yes)
 		(dnp no)
-		(property "Reference" "C5"
+		(property "Reference" "C?"
 			(at 293.116 62.484 90)
 			(effects
@@
 		(dnp no)
 		(fields_autoplaced yes)
-		(property "Reference" "#PWR026"
+		(property "Reference" "#PWR?"
 			(at 328.93 63.5 0)
 			(effects
@@
 		(dnp no)
 		(fields_autoplaced yes)
-		(property "Reference" "R8"
+		(property "Reference" "R?"
 			(at 199.39 111.7599 0)
 			(effects
@@
 		(dnp no)
 		(fields_autoplaced yes)
-		(property "Reference" "#PWR035"
+		(property "Reference" "#PWR?"
 			(at 311.15 101.6 0)
 			(effects

Commit message: I2C change
Parts:
- removed C?: 100n, Capacitor_SMD:C_0402_1005Metric, symbol Device:C
- removed R? (x2): 10k, Resistor_SMD:R_0402_1005Metric, symbol Device:R
- removed R? (x2): 4k7, Resistor_SMD:R_0402_1005Metric, symbol Device:R
- removed Y?: RV-3032-C7, rv-3032-c7:RV3032C7, symbol rv-3032-c7:RV-3032-C7
- gave numbers to parts that had none: 8
Connections:
- net +3.3V: now also U1.44 (VDD_3V3), U1.45 (VDD_3V3); no longer U1.16 (RESERVED), U1.18 (RESERVED)
- net GND: now also U1.1 (GND), U1.11 (GND), U1.17 (GND), U1.21 (GND), U1.27 (GND), U1.3 (GND), U1.34 (GND), U1.4 (GND), U1.41 (GND), U1.46 (GND), U1.49 (GND), U1.55 (GND), U1.56 (GND), U1.57 (GND), U1.58 (GND), U1.59 (GND), U1.6 (GND), U1.60 (GND), U1.61 (GND), U1.62 (GND), U1.63 (GND), U1.64 (GND), U1.65 (GND), U1.66 (GND), U1.67 (GND), U1.68 (GND), U1.69 (GND), U1.70 (GND), U1.71 (GND), U1.72 (GND), U1.73 (GND), U1.74 (GND), U1.75 (GND), U1.76 (GND), U1.77 (GND), U1.78 (GND), U1.79 (GND), U1.80 (GND), U1.81 (GND), U1.82 (GND), U1.83 (GND), U1.84 (GND), U1.85 (GND), U1.86 (GND), U1.87 (GND), U1.88 (GND), U1.89 (GND), U1.90 (GND), U1.91 (GND), U1.92 (GND), U1.93 (GND), U1.94 (GND); no longer U1.10 (TXD1), U1.12 (USB_DP), U1.13 (USB_DN), U1.14 (USB_VBUS), U1.15 (RESERVED), U1.19 (RESERVED), U1.2 (ANT_1), U1.20 (RESERVED), U1.22 (RESERVED), U1.23 (RESERVED), U1.24 (RESERVED), U1.25 (TXD2), U1.26 (NRTS2), U1.28 (NCTS2), U1.29 (RXD2), U1.30 (RESERVED), U1.31 (RESERVED), U1.32 (RESERVED), U1.33 (RESERVED), U1.35 (RESERVED), U1.36 (RESERVED), U1.37 (RESERVED), U1.38 (RESERVED), U1.39 (EVENTA), U1.40 (EVENTB), U1.42 (PPS1), U1.43 (PPS2), U1.47 (REF_O), U1.48 (REF_I), U1.5 (RESERVED), U1.50 (VREF_I), U1.51 (VREF_O), U1.52 (GPIO1), U1.53 (GPIO2), U1.54 (VANT), U1.7 (NRST_IN), U1.8 (RESERVED), U1.9 (RXD1)
- net SCL: no longer names the net of U1.30 (RESERVED)
- net SDA: no longer names the net of U1.31 (RESERVED)
- no-connect marks 6 -> 4
Other:
- note removed: "Event input not used"
- note removed: "RTC"
- note removed: "Switchover disabled"

Commit message: general clean up
Changed lines of the file:
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@@
 		(title "moTi")
 		(date "2025-09-02")
-		(rev "01")
+		(rev "02")
 		(company "Septentrio")
 		(comment 1 "Grant EUSPA/GRANT/02/2024")
@@
 		(comment 3 "co-funded by the European Union Agency for the Space ")
 		(comment 4 "moTi project has been documented by Septentrio")
+		(comment 5 "   Schematic arranged by: Laetitia.K")
 	)
 	(rectangle
@@
 		)
 	)
+	(text_box "Schematics arranged by Laetitia.K"
+		(exclude_from_sim no)
+		(at 372.11 271.78 0)
+		(size 35.56 3.9483)
+		(margins 0.9525 0.9525 0.9525 0.9525)
+		(stroke
+			(width -0.0001)
+			(type solid)
+		)
+		(fill
+			(type none)
+		)
+		(effects
+			(font
+				(size 1.27 1.27)
+				(color 132 0 0 1)
+			)
+			(justify left top)
+		)
+	)
 	(junction
 		(at 78.74 210.82)
@@
 			(project "mosaic-G5"
 				(path "/4566f719-6b00-4ec8-8709-ac6ffe4132a2"
-					(reference "D?")
+					(reference "D1")
 					(unit 1)
 				)
@@
 			(project "mosaic-G5"
 				(path "/4566f719-6b00-4ec8-8709-ac6ffe4132a2"
-					(reference "R?")
+					(reference "R1")
 					(unit 1)
 				)
@@
 			(project "mosaic-G5"
 				(path "/4566f719-6b00-4ec8-8709-ac6ffe4132a2"
-					(reference "R?")
+					(reference "R4")
 					(unit 1)
 				)
@@
 			(project "mosaic-G5"
 				(path "/4566f719-6b00-4ec8-8709-ac6ffe4132a2"
-					(reference "C?")
+					(reference "C1")
 					(unit 1)
 				)
@@
 			(project "mosaic-G5"
 				(path "/4566f719-6b00-4ec8-8709-ac6ffe4132a2"
-					(reference "J?")
+					(reference "J1")
 					(unit 1)
 				)
@@
 			(project "mosaic-G5"
 				(path "/4566f719-6b00-4ec8-8709-ac6ffe4132a2"
-					(reference "C?")
+					(reference "C2")
 					(unit 1)
 				)
@@
 			(project "mosaic-G5"
 				(path "/4566f719-6b00-4ec8-8709-ac6ffe4132a2"
-					(reference "D?")
+					(reference "D2")
 					(unit 1)
 				)
